File: sunbyte-kindlycarpet.kicad_sch (KiCad schematic)
At the start: 6 parts, among them U1 2472

Commit message: Update sunbyte-kindlycarpet.kicad_sch
Corrected LED1 and LED2 connections on the Arduino to match the 'Introduction task' example
Connections:
- net LED1: now also A1.5 (D2); no longer A1.6 (D3)
- net LED2: now also A1.6 (D3); no longer A1.5 (D2)
Changed lines of the file:
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@@
 		)
 	)
-	(label "LED1"
+	(label "LED2"
 		(at 59.69 73.66 0)
 		(effects
@@
 		)
 	)
-	(label "LED2"
+	(label "LED1"
 		(at 53.34 71.12 0)
 		(effects
